File: hardware/r4-kicad/pcb/Reid_Orthotic_v2_LHS.kicad_pcb (KiCad board)
At the start: 4 copper layers, 21.2 x 46.2 mm, 130 parts, among them J1 IO_CONN, J2 IO_CONN, J3 RF_CONN, J4 BAT_CONN, Q1 BSS816NW, Q2 DMP2110UW, Q3 RU1C002ZP, U1 LSM6DSM, U2 NRF52832-QFAA, U3 74LV4051BQ, U4 74LV4051BQ, U5 74LV4051BQ, U6 74LV4051BQ, U7 74LV4051BQ, U8 BQ24210, U9 ?TCR3UF33A,LM(CT, X1 32.768kHz NX1610SA, X2 32MHz XRCGB32M

Commit message: R4 KiCad reconstruction: schematics (LHS+RHS) + boards regenerated on fixed netlist
KiCad 7 schematic projects (PWR/MCU/MUX/IO sheets) generated from the
copper netlist with a zero-diff equivalence gate, both sides. Boards
regenerated against the MUX_VCC/castellation netlist fix (ebd13c7).
Brief: correct board outline to 21.25 x 46.25 mm (GM4 layer).

Co-Authored-By: Claude Fable 5 <noreply@anthropic.com>
Claude-Session: https://claude.ai/code/session_01VVRppXprQDNcYst2JZ14Nv
Parts:
- PAD8: value NET130 -> NET146; footprint R4:PAD_NET130_8 -> R4:PAD_NET146_8
Connections:
- net NET28 renamed NET29
- net NET33 renamed NET34
- net NET49 renamed NET50
- net NET52 renamed NET53
- net NET6 renamed NET7
- ANT1 pad 1: NET124 -> NET140
- ANT1 pad 2: NET17 -> NET18
- C16 pad 2: NET17 -> NET18
- C24 pad 2: 0V -> MUX_VCC
- C25 pad 2: 0V -> MUX_VCC
- C26 pad 2: 0V -> MUX_VCC
- C27 pad 2: 0V -> MUX_VCC
- C28 pad 2: 0V -> MUX_VCC
- C37 pad 2: NET16 -> NET17
- C38 pad 2: NET16 -> NET17
- D1 pad 1: NET16 -> NET17
- J1 pad 1: NET37 -> NET38
- J1 pad 10: NET46 -> NET47
- J1 pad 11: NET36 -> NET37
- J1 pad 12: NET58 -> NET64
- J1 pad 13: NET59 -> NET75
- J1 pad 14: NET62 -> NET78
- J1 pad 16: NET39 -> NET40
- J1 pad 17: NET40 -> NET41
- J1 pad 18: NET43 -> NET44
- J1 pad 19: NET44 -> NET45
- J1 pad 2: NET54 -> NET55
- J1 pad 3: NET61 -> NET77
- J1 pad 4: NET63 -> NET79
- J1 pad 5: NET38 -> NET39
- J1 pad 7: NET60 -> NET76
- J1 pad 8: NET41 -> NET42
- J1 pad 9: NET42 -> NET43
- J2 pad 10: 0V -> NET63
- J2 pad 11: 0V -> NET65
- J2 pad 12: 0V -> NET66
- J2 pad 13: 0V -> NET67
- J2 pad 14: 0V -> NET68
- J2 pad 15: 0V -> NET69
- J2 pad 16: 0V -> NET70
- J2 pad 17: 0V -> NET71
- J2 pad 18: 0V -> NET72
- J2 pad 19: 0V -> NET73
- J2 pad 2: 0V -> NET56
- J2 pad 20: 0V -> NET74
- J2 pad 3: 0V -> NET57
- J2 pad 4: 0V -> NET58
- J2 pad 6: 0V -> NET59
- J2 pad 7: NET55 -> NET60
- J2 pad 8: NET56 -> NET61
- J2 pad 9: NET57 -> NET62
- J3 pad 2: NET16 -> NET17
- L1 pad 1: NET103 -> NET119
- L2 pad 1: NET103 -> NET119
- L3 pad 2: NET17 -> NET18
- PAD8 pad 1: NET130 -> NET146
- Q2 pad 3: NET97 -> NET113
- Q3 pad 3: NET102 -> NET118
- R1 pad 1: NET88 -> NET104
- R10 pad 1: NET85 -> NET101
- R10 pad 2: NET38 -> NET39
- R11 pad 1: NET84 -> NET100
- R11 pad 2: NET63 -> NET79
- R12 pad 1: NET83 -> NET99
- R12 pad 2: NET62 -> NET78
- R13 pad 1: NET81 -> NET97
- R13 pad 2: NET61 -> NET77
- R14 pad 1: NET82 -> NET98
- R14 pad 2: NET60 -> NET76
- R15 pad 1: NET80 -> NET96
- R15 pad 2: NET59 -> NET75
- R16 pad 1: NET79 -> NET95
- R16 pad 2: NET58 -> NET64
- R17 pad 1: NET78 -> NET94
- R17 pad 2: NET54 -> NET55
- R18 pad 1: NET77 -> NET93
- R18 pad 2: NET37 -> NET38
- R19 pad 1: NET76 -> NET92
- R19 pad 2: NET36 -> NET37
- R2 pad 1: NET89 -> NET105
- R21 pad 2: 0V -> NET74
- R22 pad 1: NET65 -> NET81
- R22 pad 2: 0V -> NET73
- R23 pad 1: NET64 -> NET80
- R23 pad 2: 0V -> NET72
- R24 pad 2: 0V -> NET71
- R25 pad 1: NET66 -> NET82
- R25 pad 2: 0V -> NET70
- R26 pad 1: NET68 -> NET84
- R26 pad 2: 0V -> NET69
- R27 pad 1: NET67 -> NET83
- R27 pad 2: 0V -> NET68
- R28 pad 1: NET69 -> NET85
- R28 pad 2: 0V -> NET67
- R29 pad 2: 0V -> NET66
- R3 pad 1: NET94 -> NET110
- R3 pad 2: NET46 -> NET47
- R30 pad 1: NET73 -> NET89
- R30 pad 2: 0V -> NET65
- R31 pad 1: NET70 -> NET86
- R31 pad 2: 0V -> NET63
- R32 pad 1: NET71 -> NET87
- R32 pad 2: NET57 -> NET62
- R33 pad 1: NET74 -> NET90
- R33 pad 2: NET56 -> NET61
- R34 pad 2: NET55 -> NET60
- R35 pad 2: 0V -> NET59
- R36 pad 2: 0V -> NET58
- R37 pad 1: NET75 -> NET91
- R37 pad 2: 0V -> NET57
- R38 pad 1: NET72 -> NET88
- R38 pad 2: 0V -> NET56
- R4 pad 1: NET93 -> NET109
- R4 pad 2: NET44 -> NET45
- R43 pad 1: NET97 -> NET113
- R47 pad 2: 0V -> MUX_VCC
- R48 pad 2: 0V -> MUX_VCC
- R49 pad 2: 0V -> MUX_VCC
- R5 pad 1: NET92 -> NET108
- R5 pad 2: NET43 -> NET44
- R50 pad 2: 0V -> MUX_VCC
- R51 pad 2: 0V -> MUX_VCC
- R54 pad 1: 0V -> MUX_VCC
- R54 pad 2: NET102 -> NET118
- R56 pad 1: NET96 -> NET112
- R57 pad 1: NET35 -> NET36
- R58 pad 1: NET35 -> NET36
- R59 pad 1: NET100 -> NET116
- R6 pad 1: NET91 -> NET107
- R6 pad 2: NET42 -> NET43
- R7 pad 1: NET90 -> NET106
- R7 pad 2: NET41 -> NET42
- R8 pad 1: NET87 -> NET103
- R8 pad 2: NET40 -> NET41
- R9 pad 1: NET86 -> NET102
- R9 pad 2: NET39 -> NET40
- U1 pad 10: NET126 -> NET142
- U1 pad 11: NET127 -> NET143
- U1 pad 4: NET45 -> NET46
- U1 pad 9: NET125 -> NET141
- U2 pad 14: NET122 -> NET138
- U2 pad 28: NET119 -> NET135
- U2 pad 29: NET120 -> NET136
- U2 pad 37: NET45 -> NET46
- U2 pad 44: NET123 -> NET139
- U3 pad 1: NET91 -> NET107
- U3 pad 12: NET93 -> NET109
- U3 pad 13: NET113 -> NET129
- U3 pad 14: NET92 -> NET108
- U3 pad 15: NET90 -> NET106
- U3 pad 16: 0V -> MUX_VCC
- U3 pad 2: NET94 -> NET110
- U3 pad 4: NET89 -> NET105
- U3 pad 5: NET88 -> NET104
- U3 pad PAD: 0V -> MUX_VCC
- U4 pad 1: NET84 -> NET100
- U4 pad 12: NET83 -> NET99
- U4 pad 13: NET112 -> NET128
- U4 pad 14: NET82 -> NET98
- U4 pad 15: NET81 -> NET97
- U4 pad 16: 0V -> MUX_VCC
- U4 pad 2: NET87 -> NET103
- U4 pad 4: NET86 -> NET102
- U4 pad 5: NET85 -> NET101
- U4 pad PAD: 0V -> MUX_VCC
- U5 pad 1: NET78 -> NET94
- U5 pad 12: NET111 -> NET127
- U5 pad 13: NET110 -> NET126
- U5 pad 14: NET76 -> NET92
- U5 pad 15: NET77 -> NET93
- U5 pad 16: 0V -> MUX_VCC
- U5 pad 2: NET80 -> NET96
- U5 pad 4: NET79 -> NET95
- U5 pad 5: NET109 -> NET125
- U5 pad PAD: 0V -> MUX_VCC
- U6 pad 1: NET69 -> NET85
- U6 pad 12: NET108 -> NET124
- U6 pad 13: NET107 -> NET123
- U6 pad 14: NET68 -> NET84
- U6 pad 15: NET67 -> NET83
- U6 pad 16: 0V -> MUX_VCC
- U6 pad 2: NET66 -> NET82
- U6 pad 4: NET64 -> NET80
- U6 pad 5: NET65 -> NET81
- U6 pad PAD: 0V -> MUX_VCC
- U7 pad 1: NET73 -> NET89
- U7 pad 12: NET105 -> NET121
- U7 pad 13: NET106 -> NET122
- U7 pad 14: NET75 -> NET91
- U7 pad 15: NET72 -> NET88
- U7 pad 16: 0V -> MUX_VCC
- U7 pad 2: NET74 -> NET90
- U7 pad 4: NET71 -> NET87
- U7 pad 5: NET70 -> NET86
- U7 pad PAD: 0V -> MUX_VCC
- U8 pad 2: NET96 -> NET112
- U8 pad 4: NET100 -> NET116
- U8 pad 9: NET114 -> NET130
- U9 pad 3: NET35 -> NET36
- U9 pad 4: NET115 -> NET131
- X2 pad 2: NET116 -> NET132
- X2 pad 4: NET117 -> NET133
Routing:
- net 0V: track 137.6 -> 100.6 mm, vias 139 -> 127
- net MUX_VCC: track 0.00 -> 17.8 mm, vias 0 -> 12
- net NET70: track 13.6 -> 1.28 mm, vias 2 -> 0
- net NET46: track 1.35 -> 13.4 mm, vias 0 -> 2
- net NET45: track 13.4 -> 1.35 mm, vias 2 -> 0
- net NET73: track 13.1 -> 1.28 mm, vias 2 -> 0
- net NET65: track 13.0 -> 1.28 mm, vias 2 -> 0
- net NET68: track 11.5 -> 1.28 mm, vias 2 -> 0
- net NET64: track 11.5 -> 1.35 mm, vias 2 -> 0
- net NET71: track 11.1 -> 1.28 mm, vias 2 -> 0
- net NET84: track 2.26 -> 11.5 mm
- net NET81: track 3.74 -> 13.0 mm
- net NET86: track 4.78 -> 13.6 mm
- net NET67: track 10.0 -> 1.28 mm, vias 2 -> 0
- net NET80: track 3.67 -> 11.5 mm
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- added copper zone on In1.Cu, net MUX_VCC
- removed copper zone on In1.Cu, net 0V
