File: hardware/r4-kicad/pcb/Reid_Orthotic_v2_RHS.kicad_pcb (KiCad board)
At the start: 4 copper layers, 21.2 x 46.2 mm, 130 parts, among them J1 IO_CONN, J2 IO_CONN, J3 RF_CONN, J4 BAT_CONN, Q1 BSS816NW, Q2 DMP2110UW, Q3 RU1C002ZP, U1 LSM6DSM, U2 NRF52832-QFAA, U3 74LV4051BQ, U4 74LV4051BQ, U5 74LV4051BQ, U6 74LV4051BQ, U7 74LV4051BQ, U8 BQ24210, U9 ?TCR3UF33A,LM(CT, X1 32.768kHz NX1610SA, X2 32MHz XRCGB32M

Commit message: R4 KiCad reconstruction: schematics (LHS+RHS) + boards regenerated on fixed netlist
KiCad 7 schematic projects (PWR/MCU/MUX/IO sheets) generated from the
copper netlist with a zero-diff equivalence gate, both sides. Boards
regenerated against the MUX_VCC/castellation netlist fix (ebd13c7).
Brief: correct board outline to 21.25 x 46.25 mm (GM4 layer).

Co-Authored-By: Claude Fable 5 <noreply@anthropic.com>
Claude-Session: https://claude.ai/code/session_01VVRppXprQDNcYst2JZ14Nv
Connections:
- net NET14 renamed NET15
- net NET16 renamed NET17
- net NET32 renamed NET33
- net NET59 renamed NET58
- ANT1 pad 1: NET118 -> NET133
- C24 pad 2: 0V -> MUX_VCC
- C25 pad 2: 0V -> MUX_VCC
- C26 pad 2: 0V -> MUX_VCC
- C27 pad 2: 0V -> MUX_VCC
- C28 pad 2: 0V -> MUX_VCC
- J1 pad 1: NET50 -> NET51
- J1 pad 10: NET44 -> NET45
- J1 pad 11: NET100 -> NET110
- J1 pad 12: NET48 -> NET49
- J1 pad 13: NET47 -> NET48
- J1 pad 14: NET56 -> NET55
- J1 pad 16: NET38 -> NET39
- J1 pad 17: NET39 -> NET40
- J1 pad 18: NET42 -> NET43
- J1 pad 19: NET43 -> NET44
- J1 pad 2: NET49 -> NET50
- J1 pad 20: NET46 -> NET47
- J1 pad 3: NET55 -> NET54
- J1 pad 4: NET36 -> NET37
- J1 pad 5: NET37 -> NET38
- J1 pad 6: NET45 -> NET46
- J1 pad 7: NET54 -> NET53
- J1 pad 8: NET40 -> NET41
- J1 pad 9: NET41 -> NET42
- J2 pad 10: 0V -> NET103
- J2 pad 11: 0V -> NET113
- J2 pad 12: 0V -> NET97
- J2 pad 13: 0V -> NET98
- J2 pad 14: 0V -> NET114
- J2 pad 15: 0V -> NET99
- J2 pad 16: 0V -> NET115
- J2 pad 17: 0V -> NET100
- J2 pad 18: 0V -> NET101
- J2 pad 19: 0V -> NET111
- J2 pad 2: 0V -> NET52
- J2 pad 20: 0V -> NET109
- J2 pad 3: 0V -> NET108
- J2 pad 4: 0V -> NET107
- J2 pad 6: NET53 -> NET112
- J2 pad 7: NET52 -> NET106
- J2 pad 8: NET99 -> NET105
- J2 pad 9: NET51 -> NET104
- L1 pad 1: NET57 -> NET56
- L2 pad 1: NET57 -> NET56
- Q1 pad 3: NET23 -> NET24
- Q2 pad 1: NET23 -> NET24
- Q2 pad 3: NET64 -> NET63
- Q3 pad 3: NET65 -> NET64
- R1 pad 1: NET72 -> NET71
- R1 pad 2: NET46 -> NET47
- R10 pad 1: NET66 -> NET65
- R10 pad 2: NET37 -> NET38
- R11 pad 1: NET69 -> NET68
- R11 pad 2: NET36 -> NET37
- R12 pad 1: NET84 -> NET83
- R12 pad 2: NET56 -> NET55
- R13 pad 1: NET83 -> NET82
- R13 pad 2: NET55 -> NET54
- R14 pad 1: NET70 -> NET69
- R14 pad 2: NET54 -> NET53
- R15 pad 1: NET82 -> NET81
- R15 pad 2: NET47 -> NET48
- R16 pad 1: NET81 -> NET80
- R16 pad 2: NET48 -> NET49
- R17 pad 1: NET80 -> NET79
- R17 pad 2: NET49 -> NET50
- R18 pad 1: NET79 -> NET78
- R18 pad 2: NET50 -> NET51
- R19 pad 1: NET78 -> NET77
- R19 pad 2: NET100 -> NET110
- R2 pad 1: NET73 -> NET72
- R2 pad 2: NET45 -> NET46
- R21 pad 2: 0V -> NET109
- R22 pad 1: NET87 -> NET86
- R22 pad 2: 0V -> NET111
- R23 pad 1: NET88 -> NET87
- R23 pad 2: 0V -> NET101
- R24 pad 2: 0V -> NET100
- R25 pad 1: NET90 -> NET89
- R25 pad 2: 0V -> NET115
- R26 pad 1: NET91 -> NET90
- R26 pad 2: 0V -> NET99
- R27 pad 1: NET92 -> NET91
- R27 pad 2: 0V -> NET114
- R28 pad 1: NET93 -> NET92
- R28 pad 2: 0V -> NET98
- R29 pad 2: 0V -> NET97
- R3 pad 1: NET74 -> NET73
- R3 pad 2: NET44 -> NET45
- R30 pad 1: NET102 -> NET117
- R30 pad 2: 0V -> NET113
- R31 pad 1: NET75 -> NET74
- R31 pad 2: 0V -> NET103
- R32 pad 1: NET77 -> NET76
- R32 pad 2: NET51 -> NET104
- R33 pad 1: NET76 -> NET75
- R33 pad 2: NET99 -> NET105
- R34 pad 2: NET52 -> NET106
- R35 pad 2: NET53 -> NET112
- R36 pad 2: 0V -> NET107
- R37 pad 1: NET95 -> NET94
- R37 pad 2: 0V -> NET108
- R38 pad 1: NET96 -> NET95
- R38 pad 2: 0V -> NET52
- R4 pad 1: NET97 -> NET96
- R4 pad 2: NET43 -> NET44
- R42 pad 2: NET23 -> NET24
- R43 pad 1: NET64 -> NET63
- R47 pad 2: 0V -> MUX_VCC
- R48 pad 2: 0V -> MUX_VCC
- R49 pad 2: 0V -> MUX_VCC
- R5 pad 1: NET71 -> NET70
- R5 pad 2: NET42 -> NET43
- R50 pad 2: 0V -> MUX_VCC
- R51 pad 2: 0V -> MUX_VCC
- R54 pad 1: 0V -> MUX_VCC
- R54 pad 2: NET65 -> NET64
- R56 pad 1: NET63 -> NET62
- R57 pad 1: NET21 -> NET22
- R58 pad 1: NET21 -> NET22
- R59 pad 1: NET62 -> NET61
- R59 pad 2: NET22 -> NET23
- R6 pad 1: NET85 -> NET84
- R6 pad 2: NET41 -> NET42
- R60 pad 2: NET22 -> NET23
- R7 pad 1: NET98 -> NET102
- R7 pad 2: NET40 -> NET41
- R8 pad 1: NET67 -> NET66
- R8 pad 2: NET39 -> NET40
- R9 pad 1: NET68 -> NET67
- R9 pad 2: NET38 -> NET39
- U1 pad 10: NET111 -> NET126
- U1 pad 11: NET112 -> NET127
- U1 pad 9: NET110 -> NET125
- U2 pad 28: NET114 -> NET129
- U2 pad 29: NET115 -> NET130
- U2 pad 44: NET117 -> NET132
- U2 pad 9: NET113 -> NET128
- U3 pad 1: NET85 -> NET84
- U3 pad 12: NET72 -> NET71
- U3 pad 13: NET123 -> NET138
- U3 pad 14: NET73 -> NET72
- U3 pad 15: NET74 -> NET73
- U3 pad 16: 0V -> MUX_VCC
- U3 pad 2: NET98 -> NET102
- U3 pad 4: NET71 -> NET70
- U3 pad 5: NET97 -> NET96
- U3 pad PAD: 0V -> MUX_VCC
- U4 pad 1: NET69 -> NET68
- U4 pad 12: NET66 -> NET65
- U4 pad 13: NET122 -> NET137
- U4 pad 14: NET67 -> NET66
- U4 pad 15: NET68 -> NET67
- U4 pad 16: 0V -> MUX_VCC
- U4 pad 2: NET70 -> NET69
- U4 pad 4: NET83 -> NET82
- U4 pad 5: NET84 -> NET83
- U4 pad PAD: 0V -> MUX_VCC
- U5 pad 1: NET80 -> NET79
- U5 pad 12: NET119 -> NET134
- U5 pad 13: NET120 -> NET135
- U5 pad 14: NET81 -> NET80
- U5 pad 15: NET82 -> NET81
- U5 pad 16: 0V -> MUX_VCC
- U5 pad 2: NET78 -> NET77
- U5 pad 4: NET79 -> NET78
- U5 pad 5: NET121 -> NET136
- U5 pad PAD: 0V -> MUX_VCC
- U6 pad 1: NET90 -> NET89
- U6 pad 12: NET124 -> NET139
- U6 pad 13: NET125 -> NET140
- U6 pad 14: NET87 -> NET86
- U6 pad 15: NET88 -> NET87
- U6 pad 16: 0V -> MUX_VCC
- U6 pad 2: NET91 -> NET90
- U6 pad 4: NET93 -> NET92
- U6 pad 5: NET92 -> NET91
- U6 pad PAD: 0V -> MUX_VCC
- U7 pad 1: NET102 -> NET117
- U7 pad 12: NET127 -> NET142
- U7 pad 13: NET126 -> NET141
- U7 pad 14: NET77 -> NET76
- U7 pad 15: NET76 -> NET75
- U7 pad 16: 0V -> MUX_VCC
- U7 pad 2: NET96 -> NET95
- U7 pad 4: NET95 -> NET94
- U7 pad 5: NET75 -> NET74
- U7 pad PAD: 0V -> MUX_VCC
- U8 pad 2: NET63 -> NET62
- U8 pad 4: NET62 -> NET61
- U8 pad 5: NET22 -> NET23
- U8 pad 9: NET109 -> NET124
- U9 pad 3: NET21 -> NET22
- U9 pad 4: NET108 -> NET123
- X2 pad 2: NET106 -> NET121
- X2 pad 4: NET107 -> NET122
Routing:
- net 0V: track 135.7 -> 101.0 mm, vias 148 -> 136
- net MUX_VCC: track 0.00 -> 16.7 mm, vias 0 -> 12
- net NET117: track 0.00 -> 13.1 mm, vias 0 -> 2
- net NET86: track 0.00 -> 11.9 mm, vias 0 -> 2
- net NET74: track 4.39 -> 14.9 mm
- net NET89: track 0.00 -> 10.5 mm, vias 0 -> 2
- net NET88: track 10.4 -> 0.00 mm, vias 2 -> 0
- net NET102: track 13.1 -> 3.69 mm
- net NET93: track 8.39 -> 0.00 mm, vias 2 -> 0
- net NET75: track 14.9 -> 7.71 mm
- net NET97: track 7.64 -> 1.28 mm, vias 2 -> 0
- net NET77: track 10.4 -> 4.38 mm
- net NET94: track 0.00 -> 4.60 mm, vias 0 -> 2
- net NET131: track 4.58 -> 0.00 mm
- net NET96: track 3.42 -> 7.64 mm
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- added copper zone on In2.Cu, net MUX_VCC
- removed copper zone on In2.Cu, net 0V
